Commit message: mouse basic model

File: micromouse/urdf/mouse.xacro (robot description, xacro)
@@ -10,10 +10,10 @@
     <pose>0 0 0.1 0 0 0</pose>
     <inertial>
-      <mass value="15.0"/>
+      <mass value="0.0239"/>
       <origin xyz="0 0 0" rpy="0 0 0"/>
       <inertia
-          ixx="0.1" ixy="0" ixz="0"
-          iyy="0.1" iyz="0"
-          izz="0.1"
+          ixx="0.00033618" ixy="0" ixz="0"
+          iyy="0.00029902" iyz="0"
+          izz="0.00037668"
       />
     </inertial>
@@ -21,5 +21,5 @@
       <origin xyz="0 0 0" rpy="0 0 0"/>
       <geometry>
-        <box size=".4 .2 .1"/>
+        <box size=".12 .2 .05"/>
       </geometry>
     </collision>
@@ -27,5 +27,91 @@
       <origin xyz="0 0 0" rpy="0 0 0"/>
       <geometry>
-        <box size=".4 .2 .1"/>
+        <box size=".12 .2 .05"/>
+      </geometry>
+    </visual>
+    <collision name='front_caster_collision'>
+      <origin xyz="0 0.07 -0.055" rpy="0 0 0"/>
+      <geometry>
+        <sphere radius="0.03"/>
+      </geometry>
+    </collision>
+    <visual name='front_caster_visual'>
+      <origin xyz="0 0.07 -0.055" rpy="0 0 0"/>
+      <geometry>
+        <sphere radius="0.03"/>
+      </geometry>
+    </visual>
+    <collision name='rear_caster_collision'>
+      <origin xyz="0 -0.07 -0.055" rpy="0 0 0"/>
+      <geometry>
+        <sphere radius="0.03"/>
+      </geometry>
+    </collision>
+    <visual name='rear_caster_visual'>
+      <origin xyz="0 -0.07 -0.055" rpy="0 0 0"/>
+      <geometry>
+        <sphere radius="0.03"/>
+      </geometry>
+    </visual>
+  </link>
+  <joint type="continuous" name="right_wheel_joint">
+    <origin xyz="0.06 0 0" rpy="0 0 0"/>
+    <child link="right_wheel"/>
+    <parent link="base_link"/>
+    <axis xyz="1 0 0" rpy="0 0 0"/>
+    <limit effort="10000" velocity="1000"/>
+    <dynamics damping="1.0" friction="1.0"/>
+  </joint>
+  <link name='right_wheel'>
+    <inertial>
+      <mass value="0.2211"/>
+      <origin xyz="0.025 0 0" rpy="0 1.5708 0"/>
+      <inertia
+          ixx="0.01471" ixy="0" ixz="0"
+          iyy="0.01471" iyz="0"
+          izz="0.02763"
+      />
+    </inertial>
+    <collision name='collision'>
+      <origin xyz="0.025 0 0" rpy="0 1.5708 0"/>
+      <geometry>
+        <cylinder radius=".08" length=".05"/>
+      </geometry>
+    </collision>
+    <visual name='right_wheel_visual'>
+      <origin xyz="0.025 0 0" rpy="0 1.5708 0"/>
+      <geometry>
+        <cylinder radius=".08" length=".05"/>
+      </geometry>
+    </visual>
+  </link>
+  <joint type="continuous" name="left_wheel_joint">
+    <origin xyz="-0.06 0 0" rpy="0 0 0"/>
+    <child link="left_wheel"/>
+    <parent link="base_link"/>
+    <axis xyz="1 0 0" rpy="0 0 0"/>
+    <limit effort="10000" velocity="1000"/>
+    <dynamics damping="1.0" friction="1.0"/>
+  </joint>
+  <link name='left_wheel'>
+    <inertial>
+      <mass value="0.2211"/>
+      <origin xyz="-0.025 0 0" rpy="0 1.5708 0"/>
+      <inertia
+          ixx="0.01471" ixy="0" ixz="0"
+          iyy="0.01471" iyz="0"
+          izz="0.02763"
+      />
+    </inertial>
+    <collision name='collision'>
+      <origin xyz="-0.025 0 0" rpy="0 1.5708 0"/>
+      <geometry>
+        <cylinder radius=".08" length=".05"/>
+      </geometry>
+    </collision>
+    <visual name='left_wheel_visual'>
+      <origin xyz="-0.025 0 0" rpy="0 1.5708 0"/>
+      <geometry>
+        <cylinder radius=".08" length=".05"/>
       </geometry>
     </visual>

Commit message: tehetetlenségi nyomaték fix

File: micromouse/urdf/mouse.xacro (robot description, xacro)
@@ -10,10 +10,10 @@
     <pose>0 0 0.1 0 0 0</pose>
     <inertial>
-      <mass value="0.0239"/>
+      <mass value="15"/>
       <origin xyz="0 0 0" rpy="0 0 0"/>
       <inertia
-          ixx="0.00033618" ixy="0" ixz="0"
-          iyy="0.00029902" iyz="0"
-          izz="0.00037668"
+          ixx="0.1" ixy="0" ixz="0"
+          iyy="0.1" iyz="0"
+          izz="0.1"
       />
     </inertial>
@@ -65,10 +65,10 @@
   <link name='right_wheel'>
     <inertial>
-      <mass value="0.2211"/>
+      <mass value="5"/>
       <origin xyz="0.025 0 0" rpy="0 1.5708 0"/>
       <inertia
-          ixx="0.01471" ixy="0" ixz="0"
-          iyy="0.01471" iyz="0"
-          izz="0.02763"
+          ixx="0.1" ixy="0" ixz="0"
+          iyy="0.1" iyz="0"
+          izz="0.1"
       />
     </inertial>
@@ -96,10 +96,10 @@
   <link name='left_wheel'>
     <inertial>
-      <mass value="0.2211"/>
+      <mass value="5"/>
       <origin xyz="-0.025 0 0" rpy="0 1.5708 0"/>
       <inertia
-          ixx="0.01471" ixy="0" ixz="0"
-          iyy="0.01471" iyz="0"
-          izz="0.02763"
+          ixx="0.1" ixy="0" ixz="0"
+          iyy="0.1" iyz="0"
+          izz="0.1"
       />
     </inertial>

Commit message: Robot Differenciál hajtása
teleop keyboard launch file
mouse model fix

File: micromouse/urdf/mouse.xacro (robot description, xacro)
@@ -1,4 +1,5 @@
 <?xml version='1.0'?>
 <robot name="mouse" xmlns:xacro="http://www.ros.org/wiki/xacro">
+  <xacro:include filename="$(find micromouse)/urdf/mouse.gazebo" />
   <link name="base_footprint"></link>
   <joint name="base_footprint_joint" type="fixed">
@@ -21,5 +22,5 @@
       <origin xyz="0 0 0" rpy="0 0 0"/>
       <geometry>
-        <box size=".12 .2 .05"/>
+        <box size=".1 .2 .05"/>
       </geometry>
     </collision>
@@ -27,34 +28,34 @@
       <origin xyz="0 0 0" rpy="0 0 0"/>
       <geometry>
-        <box size=".12 .2 .05"/>
+        <box size=".1 .2 .05"/>
       </geometry>
     </visual>
     <collision name='front_caster_collision'>
-      <origin xyz="0 0.07 -0.055" rpy="0 0 0"/>
+      <origin xyz="0 0.07 -0.025" rpy="0 0 0"/>
       <geometry>
-        <sphere radius="0.03"/>
+        <sphere radius="0.02499"/>
       </geometry>
     </collision>
     <visual name='front_caster_visual'>
-      <origin xyz="0 0.07 -0.055" rpy="0 0 0"/>
+      <origin xyz="0 0.07 -0.025" rpy="0 0 0"/>
       <geometry>
-        <sphere radius="0.03"/>
+        <sphere radius="0.02499"/>
       </geometry>
     </visual>
     <collision name='rear_caster_collision'>
-      <origin xyz="0 -0.07 -0.055" rpy="0 0 0"/>
+      <origin xyz="0 -0.07 -0.025" rpy="0 0 0"/>
       <geometry>
-        <sphere radius="0.03"/>
+        <sphere radius="0.02499"/>
       </geometry>
     </collision>
     <visual name='rear_caster_visual'>
-      <origin xyz="0 -0.07 -0.055" rpy="0 0 0"/>
+      <origin xyz="0 -0.07 -0.025" rpy="0 0 0"/>
       <geometry>
-        <sphere radius="0.03"/>
+        <sphere radius="0.02499"/>
       </geometry>
     </visual>
   </link>
   <joint type="continuous" name="right_wheel_joint">
-    <origin xyz="0.06 0 0" rpy="0 0 0"/>
+    <origin xyz="0.05 0 0" rpy="0 0 0"/>
     <child link="right_wheel"/>
     <parent link="base_link"/>
@@ -66,5 +67,5 @@
     <inertial>
       <mass value="5"/>
-      <origin xyz="0.025 0 0" rpy="0 1.5708 0"/>
+      <origin xyz="0 0 0" rpy="0 1.5708 0"/>
       <inertia
           ixx="0.1" ixy="0" ixz="0"
@@ -76,5 +77,5 @@
       <origin xyz="0.025 0 0" rpy="0 1.5708 0"/>
       <geometry>
-        <cylinder radius=".08" length=".05"/>
+        <cylinder radius=".05" length=".05"/>
       </geometry>
     </collision>
@@ -82,10 +83,10 @@
       <origin xyz="0.025 0 0" rpy="0 1.5708 0"/>
       <geometry>
-        <cylinder radius=".08" length=".05"/>
+        <cylinder radius=".05" length=".05"/>
       </geometry>
     </visual>
   </link>
   <joint type="continuous" name="left_wheel_joint">
-    <origin xyz="-0.06 0 0" rpy="0 0 0"/>
+    <origin xyz="-0.05 0 0" rpy="0 0 0"/>
     <child link="left_wheel"/>
     <parent link="base_link"/>
@@ -97,5 +98,5 @@
     <inertial>
       <mass value="5"/>
-      <origin xyz="-0.025 0 0" rpy="0 1.5708 0"/>
+      <origin xyz="0 0 0" rpy="0 1.5708 0"/>
       <inertia
           ixx="0.1" ixy="0" ixz="0"
@@ -107,5 +108,5 @@
       <origin xyz="-0.025 0 0" rpy="0 1.5708 0"/>
       <geometry>
-        <cylinder radius=".08" length=".05"/>
+        <cylinder radius=".05" length=".05"/>
       </geometry>
     </collision>
@@ -113,5 +114,5 @@
       <origin xyz="-0.025 0 0" rpy="0 1.5708 0"/>
       <geometry>
-        <cylinder radius=".08" length=".05"/>
+        <cylinder radius=".05" length=".05"/>
       </geometry>
     </visual>

Commit message: IMU

File: micromouse/urdf/mouse.xacro (robot description, xacro)
@@ -118,3 +118,11 @@
     </visual>
   </link>
+  <!-- IMU -->
+  <joint name="imu_joint" type="fixed">
+    <origin xyz="0 0 0" rpy="0 0 0" />
+    <parent link="base_link"/>
+    <child link="imu_link" />
+  </joint>
+  <link name="imu_link">
+  </link>
 </robot>

Commit message: 2D lidar

File: micromouse/urdf/mouse.xacro (robot description, xacro)
@@ -126,3 +126,33 @@
   <link name="imu_link">
   </link>
+  <!-- Lidar -->
+  <joint type="fixed" name="scan_joint">
+    <origin xyz="0.0 0 0.06" rpy="0 0 0"/>
+    <child link="scan_link"/>
+    <parent link="base_link"/>
+    <axis xyz="0 1 0" rpy="0 0 0"/>
+  </joint>
+  <link name='scan_link'>
+    <inertial>
+      <mass value="1e-5"/>
+      <origin xyz="0 0 0" rpy="0 0 0"/>
+      <inertia
+          ixx="1e-6" ixy="0" ixz="0"
+          iyy="1e-6" iyz="0"
+          izz="1e-6"
+      />
+    </inertial>
+    <collision name='collision'>
+      <origin xyz="0 0 0.015" rpy="0 0 0"/>
+      <geometry>
+        <box size=".03 .03 .03"/>
+      </geometry>
+    </collision>
+    <visual name='scan_link_visual'>
+      <origin xyz="0 0 0.015" rpy="0 0 0"/>
+      <geometry>
+        <box size="0.03 0.03 0.03"/>
+      </geometry>
+    </visual>
+  </link>
 </robot>

Commit message: lidar tartó

File: micromouse/urdf/mouse.xacro (robot description, xacro)
@@ -53,4 +53,10 @@
       <geometry>
         <sphere radius="0.02499"/>
+      </geometry>
+    </visual>
+    <visual name='lidar_support'>
+      <origin xyz="0 0 0.04" rpy="0 0 0"/>
+      <geometry>
+        <box size=".03 .03 .04"/>
       </geometry>
     </visual>
